Commit message: camera_orientation_ok_&&tf_old_data

File: src/description/urdf/depth_camera.xacro (robot description, xacro)
@@ -4,5 +4,5 @@
         <parent link="base_link"/>
         <child link="camera_frame"/>
-        <origin xyz="0 0 0.175" rpy="0 0 0"/>
+        <origin xyz="0 0 0.3" rpy="0 0 0"/>
     </joint>
     <link name="camera_frame">
@@ -11,5 +11,26 @@
                 <cylinder radius="0.05" length="0.06"/>
             </geometry>
-            <material name="red"/>
+            <material name="blue"/>
+        </visual>
+        <collision>
+            <geometry>
+                <cylinder radius="0.05" length="0.06"/>
+            </geometry>
+        </collision>
+        <xacro:inertial_cylinder mass="0.1" length="0.06" radius="0.05">
+            <origin xyz="0 0 0" rpy="0 0 0"/>
+        </xacro:inertial_cylinder>
+    </link>
+    <joint name="camera_optical_joint" type="fixed">
+        <parent link="camera_frame"/>
+        <child link="camera_optical_link"/>
+        <origin xyz="0 0 0" rpy="-1.5707 0 -1.5707"/>
+    </joint>
+    <link name="camera_optical_link">
+        <visual>
+            <geometry>
+                <cylinder radius="0.05" length="0.06"/>
+            </geometry>
+            <material name="blue"/>
         </visual>
         <collision>
@@ -23,5 +44,5 @@
     </link>
     <gazebo reference="camera_frame">
-        <material>Gazebo/Black</material>
+        <material>Gazebo/Blue</material>
         <sensor name="camera" type="depth">
             <pose>0.064 -0.065 0.094  0 0 0 </pose>
@@ -41,5 +62,5 @@
             </camera>
             <plugin name="camera_controller" filename="libgazebo_ros_camera.so">
-                <frame_name>camera_frame</frame_name>
+                <frame_name>camera_optical_link</frame_name>
             </plugin>
         </sensor>

File: src/description/urdf/robot.urdf.xacro (robot description, xacro)
@@ -4,5 +4,5 @@
     <xacro:include filename="black_donut.xacro" />
     <!-- <xacro:include filename="gazebo_control.xacro" /> -->
-    <!-- <xacro:include filename="ros2_control.xacro" /> -->
+    <xacro:include filename="ros2_control.xacro" />
     <xacro:include filename="lidar.xacro" />
 <!--
